File: ptpe_pcb.kicad_pcb (KiCad board)
At the start: 2 copper layers, 53.8 x 71.1 mm, 11 parts, among them U1 Pico

Commit message: Somehow I forgot to upload the latest KiCAD files..
Parts:
- Misc. 1: renamed from Misc 1.
- Misc. 2: renamed from Misc 2.
- Pico1: renamed from U1; value Pico -> U1
- moved REF** 3.55 mm to (109.9, 70.8)
- moved REF** 2.70 mm to (155.2, 79.8)
- moved REF** 2.67 mm to (155.3, 77.1)
- moved Misc. 1 2.26 mm to (119.4, 118.4)
- moved Misc. 2 2.26 mm to (147.7, 118.4)
- moved Right/Up 2.26 mm to (140.6, 118.4)
- moved Select 2.26 mm to (133.5, 118.4)
- moved Left/Down 2.26 mm to (126.4, 118.4)
Connections:
- Left/Down pad 2: Net-(U1-GPIO17) -> GND
- Left/Down pad 4: Net-(U1-GPIO17) -> Net-(Pico1-GPIO17)
- Misc. 1 pad 2: Net-(U1-GPIO16) -> GND
- Misc. 1 pad 4: Net-(U1-GPIO16) -> Net-(Pico1-GPIO16)
- Misc. 2 pad 2: Net-(U1-GPIO20) -> GND
- Misc. 2 pad 4: Net-(U1-GPIO20) -> Net-(Pico1-GPIO20)
- Pico1 pad 21: Net-(U1-GPIO16) -> Net-(Pico1-GPIO16)
- Pico1 pad 22: Net-(U1-GPIO17) -> Net-(Pico1-GPIO17)
- Pico1 pad 24: Net-(U1-GPIO18) -> Net-(Pico1-GPIO18)
- Pico1 pad 25: Net-(U1-GPIO19) -> Net-(Pico1-GPIO19)
- Pico1 pad 26: Net-(U1-GPIO20) -> Net-(Pico1-GPIO20)
- Right/Up pad 2: Net-(U1-GPIO19) -> GND
- Right/Up pad 4: Net-(U1-GPIO19) -> Net-(Pico1-GPIO19)
- Select pad 2: Net-(U1-GPIO18) -> GND
- Select pad 4: Net-(U1-GPIO18) -> Net-(Pico1-GPIO18)
Routing:
- net Net-(U1-GPIO20): track 33.8 -> 0.00 mm
- net Net-(Pico1-GPIO20): track 0.00 -> 30.5 mm
- net Net-(U1-GPIO19): track 28.8 -> 0.00 mm
- net Net-(Pico1-GPIO19): track 0.00 -> 25.9 mm
- net Net-(U1-GPIO18): track 25.0 -> 0.00 mm
- net Net-(U1-GPIO17): track 22.8 -> 0.00 mm
- net Net-(Pico1-GPIO18): track 0.00 -> 21.6 mm
- net Net-(Pico1-GPIO17): track 0.00 -> 19.2 mm
- net Net-(U1-GPIO16): track 17.1 -> 0.00 mm
- net Net-(Pico1-GPIO16): track 0.00 -> 14.8 mm
- net MOSI: track 13.7 -> 17.6 mm
- net +3V3: track 49.5 -> 53.3 mm
- net +5V: track 66.7 -> 70.4 mm
- net RST: track 24.7 -> 28.1 mm
- net CS: track 50.9 -> 53.6 mm
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Other:
- board size 53.8 x 71.1 mm -> 56.2 x 71.1 mm

Commit message: Rev 2
Parts:
- Misc1: renamed from Misc. 1
- Misc2: renamed from Misc. 2
- renumbered Pico1 to Pico
Connections:
- Left/Down pad 2: GND -> unconnected-(Left/Down1-Pad2)
- Misc1 pad 2: GND -> unconnected-(Misc1-Pad2)
- Misc1 pad 3: GND -> unconnected-(Misc1-Pad3)
- Misc2 pad 2: GND -> unconnected-(Misc2-Pad2)
- Misc2 pad 3: GND -> unconnected-(Misc2-Pad3)
- Right/Up pad 2: GND -> unconnected-(Right/Up1-Pad2)
- Right/Up pad 3: GND -> unconnected-(Right/Up1-Pad3)
- Select pad 2: GND -> unconnected-(Select1-Pad2)
