File: ptpe_pcb.kicad_sch (KiCad schematic)
At the start: 6 parts, among them SW1 1825910-6, SW2 1825910-6, SW3 1825910-6, SW4 1825910-6, SW5 1825910-6, U1 Pico

Commit message: Somehow I forgot to upload the latest KiCAD files..
Parts:
- Pico1: renamed from U1; value Pico -> U1
- renumbered SW2 to Left/Down1, SW1 to Misc1, SW5 to Misc2, SW3 to Right/Up1, SW4 to Select1
Connections:
- net GND: now also Left/Down1.2, Misc1.2, Misc2.2, Right/Up1.2, Select1.2
- net at Misc1.4, Pico1.21 (GPIO16): no longer Misc1.2
- net at Left/Down1.4, Pico1.22 (GPIO17): no longer Left/Down1.2
- net at Pico1.24 (GPIO18), Select1.4: no longer Select1.2
- net at Pico1.25 (GPIO19), Right/Up1.4: no longer Right/Up1.2
- net at Misc2.4, Pico1.26 (GPIO20): no longer Misc2.2

Commit message: Rev 2
Connections:
- net GND: no longer Left/Down1.2, Misc1.2, Misc1.3, Misc2.2, Misc2.3, Right/Up1.2, Right/Up1.3, Select1.2
